File: PCB/guilty-devboard-idk.kicad_sch (KiCad schematic)
At the start: 62 parts, among them J1 USB_C_Receptacle_USB2.0_14P, J3 Mirrored TCA9535 pads, Q1 SP2038CNQ, Q2 Q_PMOS, SW1 SW_Push, U1 nRF52840-CKXX, U2 SGM40567-4.2XG/TR, U3 DW01A, U4 MIC2876-5.0YMT-TR, U5 AD5274BCPZ-100-RL7, U6 AW13412HDNR, U7 TPS63031DSK, U8 Xiao nRF52840 Connectors, Y1 32MHz

Commit message: commit idk pre-10.0 update
Parts:
- removed AE2: Antenna, Connector_Coaxial:U.FL_Molex_MCRF_73412-0110_Vertical, symbol Device:Antenna
- removed U1: nRF52840-CKXX, PCM_nordic-lib-kicad-nrf52:BGA-94_10x10_3.544x3.607mm, symbol PCM_nordic-lib-kicad-nrf52:nRF52840-CKXX
- removed U6: AW13412HDNR, easyeda2kicad:TSNP-6_L1.1-W0.7-P0.40-BL, symbol easyeda2kicad:AW13412HDNR
- added C23: 4.7uF, Capacitor_SMD:C_0201_0603Metric, symbol Device:C
- added C24, C25: DNP, Capacitor_SMD:C_0201_0603Metric, symbol Device:C
- added U1: nRF52840-QIXX, Package_DFN_QFN:Nordic_AQFN-73-1EP_7x7mm_P0.5mm, symbol PCM_nordic-lib-kicad-nrf52:nRF52840-QIXX
- C1: value 820pF -> 100pF
- C4: value 4.7uF -> 820pF
- R13: footprint (none) -> Resistor_SMD:R_0201_0603Metric
Connections:
- net +3V3: now also U1.A22 (VDD), U1.AD14 (VDD), U1.AD23 (VDD), U1.B1 (VDD), U1.W1 (VDD), U1.Y2 (VDDH)
- net 5V_BOOST_ENABLE: now also U1.A14 (P1.15)
- net 5V_POWER_GOOD: now also U1.A16 (P1.13)
- net AGND: now also C23.2, C24.2, C25.2, U1.A23 (XC2), U1.B24 (XC1), U1.B7 (VSS), U1.EP (VSS), U1.F23 (VSS_PA)
- net ANT: now also AE1.2 (PCB_Trace)
- net BATT_LEVEL: now also U1.A8 (P0.31)
- net CHARGE_STATUS: now also U1.B15 (P1.14)
- net DCC: now also C25.1, U1.B3 (DCC), U1.B5 (DEC4), U1.E24 (DEC6)
- net I2C_SCL: now also U1.N1 (P0.08)
- net I2C_SDA: now also U1.L1 (P0.06)
- net P0.02_AIN0: now also U1.A12 (P0.02)
- net P0.03_AIN1: now also U1.B13 (P0.03)
- net P0.04_AIN2: now also U1.J1 (P0.04)
- net P0.05_AIN3: now also U1.K2 (P0.05)
- net RESET: now also U1.AC13 (~{RESET})
- net SWDCLK: now also U1.AA24 (SWDCLK)
- net SWDIO: now also U1.AC24 (SWDIO)
- net VBUS: now also U1.AD2 (VBUS)
- net at C1.1: now also U1.D23 (DEC3)
- net at C4.1: now also U1.N24 (DEC5)
- net at C5.2: now also U1.C1 (DEC1)
- net at L4.1: now also U1.H23 (ANT)
- net at R5.2: now also U1.AD4 (D-)
- net at R4.2: now also U1.AD6 (D+)
- new net: C23.1, U1.AC5 (DECUSB)
- new net: C24.1, U1.A18 (DEC2)
- no-connect marks 1 -> 2
Other:
- note added: "antenna"
- note added: "todo: - check pin assignments match with CKAA - add the rest of the gpio - pcb it - double check DCC/DEC4/6 routing - make sure to route VSS_PA to C3 (ANT) GND"
- note removed: "antennas"
- note removed: "todo: - add the rest of the gpio - make sure to route VSS_PA to C3 (ANT) GND - pcb it"
- moved on the sheet: AE1, C1, C12, C16, C2, C21, C3, C4, C5, J1, J3, L1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

Commit message: update idk schematic is done aside from switching out 3.3V
Parts:
- removed AE1: Antenna_Chip, RF_Antenna:Johanson_2450AT18x100_2400-2500Mhz, symbol Device:Antenna_Chip
- removed C1: 100pF, Capacitor_SMD:C_0201_0603Metric, symbol Device:C
- removed C10, C12, C23: 4.7uF, Capacitor_SMD:C_0201_0603Metric, symbol Device:C
- removed C11, C13: 8.0pF, Capacitor_SMD:C_0201_0603Metric, symbol Device:C
- removed C2, C6: 1.0uF, Capacitor_SMD:C_0201_0603Metric, symbol Device:C
- removed C24, C25: DNP, Capacitor_SMD:C_0201_0603Metric, symbol Device:C
- removed C4: 820pF, Capacitor_SMD:C_0201_0603Metric, symbol Device:C
- removed C5, C7, C8, C9: 100nF, Capacitor_SMD:C_0201_0603Metric, symbol Device:C
- removed D1: D, Diode_SMD:D_SOD-882, symbol Device:D
- removed R10, R11, R3: 10k, Resistor_SMD:R_0201_0603Metric, symbol Device:R
- removed R7: 470, Resistor_SMD:R_0201_0603Metric, symbol Device:R
- removed U1: nRF52840-QIXX, Package_DFN_QFN:Nordic_AQFN-73-1EP_7x7mm_P0.5mm, symbol PCM_nordic-lib-kicad-nrf52:nRF52840-QIXX
- removed U3: DW01A, Package_TO_SOT_SMD:SOT-23-6, symbol Battery_Management:DW01A
- removed U5: AD5274BCPZ-100-RL7, easyeda2kicad:LFCSP-10_L3.0-W3.0-P0.50-BL-EP, symbol easyeda2kicad:AD5274BCPZ-100-RL7
- removed U8: Xiao nRF52840 Connectors, guilty-devboard-idk:Xiao nRF52840 pads, symbol guilty-devboard:Xiao nRF52840 Connectors
- added AE1: Antenna_Chip, symbol KiCad:Antenna_Chip
- added C1: 10uF, symbol KiCad:C_Small
- added C10, C11, C4: 4.7uF, symbol KiCad:C_Small
- added C12: 0.1uF, symbol KiCad:C_Small
- added C13, C6: 2.2uF, symbol KiCad:C_Small
- added C2, C8, C9: 100nF, symbol KiCad:C_Small
- added C5: 1.0pF, symbol KiCad:C_Small
- added C7: DNP, symbol KiCad:C_Small
- added FB1: FerriteBead, symbol KiCad:FerriteBead_Small
- added L5: 3.6nH, Inductor_SMD:L_0201_0603Metric, symbol Device:L
- added L6: 4.7uH, symbol KiCad:L_Small
- added L7: 1.0nH, symbol KiCad:L_Small
- added R14: 220k, symbol KiCad:R_Small
- added R15: 68k, symbol KiCad:R_Small
- added R16: 2.2, symbol KiCad:R_Small
- added R17: 200, Resistor_SMD:R_0201_0603Metric, symbol Device:R
- added R18: 1M, Resistor_SMD:R_0201_0603Metric, symbol Device:R_Small
- added R3: 470k, symbol KiCad:R_Small
- added R7: 1k, symbol KiCad:R_Small
- added U1: nRF54LM20A-PAXX, PCM_nordic-lib-kicad-nrf54l:Nordic_FCCSP-98_3.67x3.85mm_Layout10x10_P0.35mm_Offcenter, symbol PCM_nordic-lib-kicad-nrf54l:nRF54LM20A-PAXX
- added U3: Xiao nRF52840 Connectors, guilty-devboard-idk:Xiao nRF52840 pads, symbol guilty-devboard:Xiao nRF52840 Plus Connectors
- added U5: FH9261-G3JH, Package_TO_SOT_SMD:SOT-23-6, symbol guilty-devboard:FH9261-G3JH
- added Y2: 32.768kHz, Crystal:Crystal_SMD_2016-4Pin_2.0x1.6mm, symbol Device:Crystal
- C15: value 0.1uF -> 1.5pF
- C17: value 0.1uF -> 4.7uF
- C18: value 1uF -> 1.5pF
- C3: value 1.0pF -> DNP
- L1: value 4.7nH -> 3.3nH
- L4: value 3.9nH -> 4.7nH
Connections:
- net +3V3: now also C1.1, C2.1, C8.1, C9.1, U1.A3 (VDD), U1.A4 (VDD), U1.A9 (VDD), U1.G10 (VDD), U1.H1 (VDD), U3.10 (3V3); no longer C17.2, U2.B2 (nCHG)
- net +5V: now also U3.8 (5V)
- net +BATT: now also C17.1, U2.A1 (BAT), R7.1, U3.24 (BAT+)
- net -BATT: now also C12.2, U3.25 (BAT-), U5.6 (VSS); no longer C15.1
- net 5V_BOOST_ENABLE: now also U1.D4 (P3.12)
- net 5V_POWER_GOOD: now also R18.1, U1.E4 (P3.11); no longer R13.1, U4.7 (/PG)
- net AGND: now also C15.1, C17.2, C1.2, C10.1, C11.2, C13.1, C2.2, C4.2, C6.2, C7.2, C8.2, C9.2, R17.1, R3.2, U1.A1 (VSS), U1.A10 (VSS), U1.A7 (VSS), U1.D1 (VSS), U1.D2 (VSS), U1.E5 (VSS), U1.E6 (VSS), U1.F1 (VSS), U1.F5 (VSS), U1.F6 (VSS), U1.K1 (VSS), U1.K10 (VSS), U3.29 (GND), U3.9 (GND); no longer C17.1, U2.C1 (IREF), Y1.1, Y1.2
- net ANT: now also L5.1, U1.E1 (ANT); no longer L1.2
- net BATT_LEVEL: now also U1.K8 (P1.00)
- net CHARGE_STATUS: now also U2.B2 (nCHG), U1.F4 (P3.10)
- net I2C_SCL: now also J3.15 (SCL), U3.6 (A/D5_SCL)
- net I2C_SDA: now also J3.14 (SDA), U3.5 (A/D4_SDA)
- net RESET: now also U1.F2 (~{RESET}), U3.28 (RST)
- net SWDCLK: now also U1.G1 (SWDCLK), U3.27 (CLK)
- net SWDIO: now also U1.G2 (SWDIO), U3.26 (DIO)
- net VBUS: now also R16.1
- net at Q1.2 (G1): now also U5.1 (DO)
- net at R6.1: now also U5.2 (VM)
- net at Q1.5 (G2): now also U5.3 (CO)
- net at C15.2: now also L1.1, L4.2
- net at C22.2, L2.1, Q2.S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: now also C10.2
- net at C18.2: now also L4.1, L5.2
- net at R5.2: now also U1.K4 (D-)
- net at R4.2: now also U1.K5 (D+)
- new net: R14.1, R15.1, R3.1, U2.C1 (IREF)
- new net: U1.A2 (XC1), Y1.2
- new net: L6.1, U1.A5 (DCC)
- new net: C4.1, FB1.1, L6.2, U1.A6 (DECD)
- new net: C5.1, C6.1, C7.1, FB1.2, L7.2, U1.A8 (DECA)
- new net: U1.B1 (XC2), Y1.1
- new net: C5.2, L7.1, U1.C1 (DECRF)
- new net: U1.C6 (P1.20), Y2.2
- new net: U1.C7 (P1.21), Y2.1
- new net: R17.2, U1.J5 (TXRTUNE)
- new net: C13.2, U1.K6 (DECUSB)
- new net: C11.1, R16.2, U1.K7 (VBUS)
- new net: R13.1, R18.2, U4.7 (/PG)
- new net: AE1.1 (FEED), C3.2, L1.2
- new net: C12.1, R7.2, U5.5 (VDD)
- new net FAST_CHARGE_1: R14.2, U1.G4 (P3.08)
- new net FAST_CHARGE_2: R15.2, U1.F7 (P3.09)
- new net P1.01_NFC1: U3.18 (D14_NFC1)
- new net P1.02_NFC2: U3.19 (D15_NFC2)
- no-connect marks 2 -> 1
Other:
- note added: "Antenna"
- note added: "Battery"
- note added: "Notes if VDDH is applied and >VDD, high voltage mode is used otherwise, connect VDD to VDDH hence here it runs in low voltage mode potential power savings: - PMOS for voltage divider (1uA)? - make voltage divider more efficient? - remove voltage divider entirely? - boards using original xiao will need a separate one anyways, and this allows for easier testing of different resistor values to see w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"
- note added: "Reset circuitry Perhaps unnecessary, can be more basic if need be"
- note added: "TODO: - add the rest of the gpio - does the other end of the antenna need GND? idk - pcb it - double check decoupling routing - make sure to place crystals and antenna filter as close as possible to MCU - crystals can be far but that requires adjusting load capacitance and calculating trace capacitance is a huge pain"
- note added: "TODO: check power savings"
- note added: "TODO: connect io thingies"
- note added: "TODO: maybe add an easier to access alternative swd pins?"
- note added: "analog"
- note added: "digital"
- note added: "gpio goes hereeeeeeeeeeeeeeee (and right)"
- note added: "sink neither for 51mA sink 1 for 160mA sink 2 for 400mA sink both for 500mA"
- note removed: "B3"
- note removed: "B8"
- note removed: "Battery pads"
- note removed: "DEC4/6/DCC decoupling"
- note removed: "K1"
- note removed: "K5"
- note removed: "Notes if VDDH is applied and >VDD, high voltage mode is used otherwise, connect VDD to VDDH hence here it runs in low voltage mode potential power savings: - 32.768k crystal (1uA) - PMOS for voltage divider (<1uA) not worth the space used for miniscule power savings - maybe check for higher efficiency 3.3v regulators? - maybe remove 5V_PG - maybe add recommended VIN cap near 5V reg"
- note removed: "TODO: switch to nrf52840 plus clone still working on that symbol and footprint (also connect the rest of the GPIO lol)"
- note removed: "VDD decoupling/capacitors/idk"
- note removed: "antenna"
- note removed: "digipot (digital rheostat) to control battery charging current"
- note removed: "gpio goes hereeeeeeeeeeeeeeee"
- note removed: "i2c pullups"
- note removed: "maybe add an easier to access swdio/swdclk thing? at least if there's space"
- note removed: "todo: - check pin assignments match with CKAA - add the rest of the gpio - pcb it - double check DCC/DEC4/6 routing - make sure to route VSS_PA to C3 (ANT) GND"
- moved on the sheet: C14, C16, C19, C20, C21, C22, C3, D2, D3, D4, D5, D6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

Commit message: idk pretty much finish schematic everything should be right, besides adding more basic gpio when convenient
Parts:
- removed L3: 1.5uH, Inductor_SMD:L_0402_1005Metric, symbol Device:L
- removed U7: TPS63031DSK, Package_SON:WSON-10-1EP_2.5x2.5mm_P0.5mm_EP1.2x2mm, symbol Regulator_Switching:TPS63031DSK
- added C23: 0.47uF, symbol KiCad:C_Small
- added L3: 1.5uH, symbol KiCad:L_Small
- added U6: BD83070GWL-E2, guilty-devboard-idk:BD83070GWL, symbol guilty-devboard:BD83070GWL-E2
Connections:
- net I2C_SCL is gone; now on net P1.31_A/D5_I2C_SCL: J3.15 (SCL), U3.6 (A/D5_SCL)
- net I2C_SDA is gone; now on net P1.30_A/D4_I2C_SDA: J3.14 (SDA), U3.5 (A/D4_SDA)
- net +3V3: now also U6.B1 (FB), U6.C1 (VOUT)
- net AGND: now also C23.2, U6.A2 (GND), U6.B2 (MODE), U6.D2 (PGND)
- net P1.01_NFC1: now also U1.J6 (P1.01)
- net P1.02_NFC2: now also U1.J7 (P1.02)
- net P2.00_QSPI.D3_SPIM.DCX: now reaches U1.B10 (P2.00)
- net P2.00_QSPI.D3_SPIM.DCX: now also U3.22 (D18_MISO1)
- net P2.01_QSPI/SPIM.SCK: now reaches U1.C10 (P2.01)
- net P2.01_QSPI/SPIM.SCK: now also U3.13 (D8_SCK)
- net P2.07_UARTE00.RXD: now reaches U1.C9 (P2.07)
- net P2.07_UARTE00.RXD: now also U3.14 (D7_RX)
- net P2.02_QSPI.D0-SPIM.MOSI/SDO: now reaches U1.D10 (P2.02)
- net P2.02_QSPI.D0-SPIM.MOSI/SDO: now also U3.11 (D10_MOSI)
- net P2.08_UARTE00.TXD: now reaches U1.D9 (P2.08)
- net P2.08_UARTE00.TXD: now also U3.7 (D6_TX)
- net P2.03_QSPI.D2: now reaches U1.E10 (P2.03)
- net P2.03_QSPI.D2: now also U3.21 (D19_MOSI1)
- net P2.09_UARTE00.CTS: now reaches U1.E9 (P2.09)
- net P2.09_UARTE00.CTS: now also U3.15 (D11)
- net P2.04_QSPI.D1-SPIM.MISO/SDI: now reaches U1.F10 (P2.04)
- net P2.04_QSPI.D1-SPIM.MISO/SDI: now also U3.12 (D9_MISO)
- net P2.10_UARTE00.RTS: now reaches U1.F9 (P2.10)
- net P2.10_UARTE00.RTS: now also U3.16 (D12)
- net P2.05_QSPI.CSN: now reaches U1.G9 (P2.05)
- net P2.05_QSPI.CSN: now also U3.23 (D17_SCK1)
- net at D6.1 (K), D7.1 (K): now also U6.A1 (EN), U6.B3 (VIN), U6.C2 (VSEL), U6.C3 (PVIN)
- net P1.07_GRTC.CLKOUTFAST: now reaches U1.G8 (P1.07)
- net P1.07_GRTC.CLKOUTFAST: now also J3.8 (P01)
- net P1.29_D16_A6: now reaches U1.H10 (P1.29)
- net P1.29_D16_A6: now also U3.20 (D16_A6)
- net P1.05_A/D2: now reaches U1.H8 (P1.05)
- net P1.05_A/D2: now also U3.3 (A/D2)
- net P1.03_A/D0: now reaches U1.H9 (P1.03)
- net P1.03_A/D0: now also U3.1 (A/D0)
- net P1.30_A/D4_I2C_SDA: now reaches U1.J10 (P1.30)
- net P1.06_A/D3: now reaches U1.J8 (P1.06)
- net P1.06_A/D3: now also U3.4 (A/D3)
- net P1.04_A/D1: now reaches U1.J9 (P1.04)
- net P1.04_A/D1: now also U3.2 (A/D1)
- net P1.31_A/D5_I2C_SCL: now reaches U1.K9 (P1.31)
- net P0.04_GRTC.CLKOUT32K: now reaches J3.9 (P00)
- net P0.04_GRTC.CLKOUT32K: now also U1.J1 (P0.04)
- net P0.03_GRTC.PWM: now reaches U3.17 (D13)
- net P0.03_GRTC.PWM: now also U1.J2 (P0.03)
- new net: L3.1, U6.D3 (LX1)
- new net: L3.2, U6.D1 (LX2)
- new net: C23.1, U6.A3 (REF)
Other:
- note added: "Notes if VDDH is applied and >VDD, high voltage mode is used otherwise, connect VDD to VDDH hence here it runs in low voltage mode potential power savings: - make voltage divider more efficient? - remove voltage divider entirely? - boards using original xiao will need a separate one anyways, and this allows for easier testing of different resistor values to see what works"
- note added: "TODO: - add the rest of the gpio - does the other end of the antenna need GND? idk - pcb it - double check decoupling routing - make sure to place crystals and antenna filter as close as possible to MCU - crystals can be far but that requires adjusting load capacitance and calculating trace capacitance is a huge pain - do fancy antennas stuff ofc (impedance match everything to 50 ohms) - add basi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"
- note removed: "Notes if VDDH is applied and >VDD, high voltage mode is used otherwise, connect VDD to VDDH hence here it runs in low voltage mode potential power savings: - PMOS for voltage divider (1uA)? - make voltage divider more efficient? - remove voltage divider entirely? - boards using original xiao will need a separate one anyways, and this allows for easier testing of different resistor values to see w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"
- note removed: "TODO: - add the rest of the gpio - does the other end of the antenna need GND? idk - pcb it - double check decoupling routing - make sure to place crystals and antenna filter as close as possible to MCU - crystals can be far but that requires adjusting load capacitance and calculating trace capacitance is a huge pain"
- note removed: "TODO: connect io thingies"
- note removed: "TODO: maybe add an easier to access alternative swd pins?"
- note removed: "analog"
- note removed: "digital"
- moved on the sheet: C19, D6, D7, J3

Commit message: terrible half done routing idk - post-decent filter routing
Parts:
- removed J1: USB_C_Receptacle_USB2.0_14P, Connector_USB:USB_C_Receptacle_HRO_TYPE-C-31-M-12, symbol Connector:USB_C_Receptacle_USB2.0_14P
- removed J3: Mirrored TCA9535 pads, Package_SO:TSSOP-24_4.4x7.8mm_P0.65mm, symbol guilty-devboard:Mirrored TCA9535PWR pads
- removed SW1: SW_Push, symbol Switch:SW_Push
- removed U3: Xiao nRF52840 Connectors, guilty-devboard-idk:Xiao nRF52840 pads, symbol guilty-devboard:Xiao nRF52840 Plus Connectors
- removed Y1: 32MHz, Crystal:Crystal_SMD_2016-4Pin_2.0x1.6mm, symbol Device:Crystal
- removed Y2: 32.768kHz, Crystal:Crystal_SMD_2016-4Pin_2.0x1.6mm, symbol Device:Crystal
- added J1: USB_C_Receptacle_USB2.0_16P, Connector_USB:USB_C_Receptacle_Amphenol_124019772112A, symbol KiCad:USB_C_Receptacle_USB2.0_16P
- added JP2: Jumper_2_Bridged, Resistor_SMD:R_0201_0603Metric, symbol KiCad:Jumper_2_Bridged
- added U3: Xiao nRF52840 Connectors, guilty-devboard-idk:Guilty Devboard Xrd pads, symbol guilty-devboard:Guilty Devboard Xrd Connectors (dev)
- added Y1: 32MHz, Crystal:Crystal_SMD_2016-4Pin_2.0x1.6mm, symbol KiCad:Crystal_GND24
- added Y2: 32.768kHz, Crystal:Crystal_SMD_2016-4Pin_2.0x1.6mm, symbol KiCad:Crystal_GND24
- AE1: footprint (none) -> PCM_marbastlib-various:2450AT18D0100001E_L
- C1, C10, C11, C12, C13, C2, C23, C4, C5, C6, C7, C8, C9: footprint (none) -> Capacitor_SMD:C_0201_0603Metric
- C16, C19, C20: footprint Capacitor_SMD:C_0402_1005Metric -> Capacitor_SMD:C_0201_0603Metric
- C18: value 1.5pF -> 1.2pF
- D4: footprint Diode_SMD:D_SOD-123 -> Diode_SMD:D_SOD-323
- D5: footprint guilty-devboard-idk:0603_DSN_AND8464-D -> Diode_SMD:D_SOD-323
- D6: footprint guilty-devboard-idk:0603_DSN_AND8464-D -> Diode_SMD:D_SOD-882
- FB1, L3, L6, L7: footprint (none) -> Inductor_SMD:L_0201_0603Metric
- L2: footprint Inductor_SMD:L_0402_1005Metric -> Inductor_SMD:L_0201_0603Metric
- Q2: footprint Inductor_SMD:L_0603_1608Metric -> guilty-devboard-idk:Vishay_PowerPAK_SC70-6L_Single
- R14, R15, R16, R3, R7: footprint (none) -> Resistor_SMD:R_0201_0603Metric
- R8: footprint Resistor_SMD:R_0402_1005Metric -> Resistor_SMD:R_0201_0603Metric
Connections:
- net +3V3: now also U3.10 (3V3), U3.34 (V_{DD}), U3.43 (RESET), U3.58 (EP)
- net +5V: now also U3.8 (5V)
- net +BATT: now also U3.24 (BAT+)
- net -BATT: now also U3.25 (BAT-)
- net P0.03_GRTC.PWM: now also U3.17 (D13)
- net P0.04_GRTC.CLKOUT32K: now also U3.46 (GP_{A}0)
- net P1.01_NFC1: now also U3.18 (D14_NFC1)
- net P1.02_NFC2: now also U3.19 (D15_NFC2)
- net P1.03_A/D0: now also U3.1 (A/D0)
- net P1.04_A/D1: now also U3.2 (A/D1)
- net P1.05_A/D2: now also U3.3 (A/D2)
- net P1.06_A/D3: now also U3.4 (A/D3)
- net P1.07_GRTC.CLKOUTFAST: now also U3.47 (GP_{A}1)
- net P1.29_D16_A6: now also U3.20 (D16_A6)
- net P1.30_A/D4_I2C_SDA: now also U3.38 (SDA), U3.5 (A/D4_SDA)
- net P1.31_A/D5_I2C_SCL: now also U3.37 (SCL), U3.6 (A/D5_SCL)
- net P2.00_QSPI.D3_SPIM.DCX: now also U3.22 (D18_MISO1)
- net P2.01_QSPI/SPIM.SCK: now also U3.13 (D8_SCK)
- net P2.02_QSPI.D0-SPIM.MOSI/SDO: now also U3.11 (D10_MOSI)
- net P2.03_QSPI.D2: now also U3.21 (D19_MOSI1)
- net P2.04_QSPI.D1-SPIM.MISO/SDI: now also U3.12 (D9_MISO)
- net P2.05_QSPI.CSN: now also U3.23 (D17_SCK1)
- net P2.07_UARTE00.RXD: now also U3.14 (D7_RX)
- net P2.08_UARTE00.TXD: now also U3.7 (D6_TX)
- net P2.09_UARTE00.CTS: now also U3.15 (D11)
- net P2.10_UARTE00.RTS: now also U3.16 (D12)
- net RESET: now also JP2.1 (A), U3.28 (RST)
- net SWDCLK: now also U3.27 (CLK)
- net SWDIO: now also U3.26 (DIO)
- net USB_D+: now also J1.A6 (D+), J1.B6 (D+)
- net USB_D-: now also J1.A7 (D-), J1.B7 (D-)
- net VBUS: now also J1.A4 (VBUS), J1.A9 (VBUS), J1.B4 (VBUS), J1.B9 (VBUS)
- net at U1.A2 (XC1): now also Y1.1
- net at U1.B1 (XC2): now also Y1.3
- net at U1.C6 (P1.20): now also Y2.1
- net at U1.C7 (P1.21): now also Y2.3
- net at R1.1: now also J1.A5 (CC1)
- net at R2.1: now also J1.B5 (CC2)
- net P1.15: now reaches U1.B2 (P1.15)
- net P1.15: now also U3.55 (GP_{B}1)
- net P1.16: now reaches U1.B3 (P1.16)
- net P1.16: now also U3.56 (GP_{B}2)
- net P1.17: now reaches U1.B4 (P1.17)
- net P1.17: now also U3.57 (GP_{B}3)
- net P1.18: now reaches U1.B5 (P1.18)
- net P1.18: now also U3.30 (GP_{B}4)
- net P1.19: now reaches U1.B6 (P1.19)
- net P1.19: now also U3.31 (GP_{B}5)
- net P1.23: now reaches U1.B7 (P1.23)
- net P1.23: now also U3.33 (GP_{B}7)
- net MCP23017_A0: now reaches U1.B8 (P1.26)
- net MCP23017_A0: now also U3.40 (A0)
- net P1.14: now reaches U1.C2 (P1.14)
- net P1.14: now also U3.54 (GP_{B}0)
- net P1.13: now reaches U1.C3 (P1.13)
- net P1.13: now also U3.53 (GP_{A}7)
- net P1.12: now reaches U1.C4 (P1.12)
- net P1.12: now also U3.52 (GP_{A}6)
- net P1.11: now reaches U1.C5 (P1.11)
- net P1.11: now also U3.51 (GP_{A}5)
- net MCP23017_A1: now reaches U1.C8 (P1.27)
- net MCP23017_A1: now also U3.41 (A1)
- net P1.10: now reaches U1.D5 (P1.10)
- net P1.10: now also U3.50 (GP_{A}4)
- net P1.22: now reaches U1.D6 (P1.22)
- net P1.22: now also U3.32 (GP_{B}6)
- net MCP23017_INTA: now reaches U1.D7 (P1.24)
- net MCP23017_INTA: now also U3.45 (INT_{A})
- net MCP23017_A2: now reaches U1.D8 (P1.28)
- net MCP23017_A2: now also U3.42 (A2)
- net MCP23017_INTB: now reaches U1.E7 (P1.25)
- net MCP23017_INTB: now also U3.44 (INT_{B})
- net P1.09: now reaches U1.E8 (P1.09)
- net P1.09: now also U3.49 (GP_{A}3)
- net P1.08: now reaches U1.F8 (P1.08)
- net P1.08: now also U3.48 (GP_{A}2)
- net AGND renamed GND
- net GND: now also J1.A1 (GND), J1.A12 (GND), J1.B1 (GND), J1.B12 (GND), J1.SH (SHIELD), JP2.2 (B), U3.29 (GND), U3.35 (V_{SS}), U3.9 (GND), Y1.2 (G), Y1.4 (G), Y2.2 (G), Y2.4 (G)
- no-connect marks 1 -> 0
Other:
- note added: "AGND would be AGND (connected to GND at *one* point) but this is the only thing using AGND so just connecting it to GND directly"
- note added: "Notes potential power savings: - make voltage divider more efficient? - remove voltage divider entirely? - boards using original xiao will need a separate one anyways, and this allows for easier testing of different resistor values to see what works"
- note added: "TODO: when wiring rear GPIO, wire INTa/b and addresses (if possible) to GPIO too!!!"
- note removed: "AGND and GND should be connected at one spot"
- note removed: "AGND-GND"
- note removed: "Notes if VDDH is applied and >VDD, high voltage mode is used otherwise, connect VDD to VDDH hence here it runs in low voltage mode potential power savings: - make voltage divider more efficient? - remove voltage divider entirely? - boards using original xiao will need a separate one anyways, and this allows for easier testing of different resistor values to see what works"
- moved on the sheet: C10, C20, C22, D2, D3, D4, D5, L2, Q2, R1, R13, R18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
